Commit message: Rename demo_tb3 pkg to demo_tb3_urdf
Signed-off-by: C88-YQ <1409947012@qq.com>

File: ns_support_demo/demo_tb3_urdf/urdf/gz_waffle.sdf.xacro (robot description, xacro)
@@ -2,5 +2,5 @@
 <sdf version="1.6" xmlns:xacro="http://www.ros.org/wiki/xacro">
     <xacro:arg name="namespace" default=""/>
-    <model name="turtlebot3_waffle_gps">
+    <model name="turtlebot3_waffle">
       <pose>0.0 0.0 0.0 0.0 0.0 0.0</pose>
       <link name="base_footprint"/>
@@ -30,5 +30,5 @@
           <geometry>
             <mesh>
-              <uri>package://demo_tb3/models/turtlebot3_model/meshes/waffle_base.dae</uri>
+              <uri>package://demo_tb3_urdf/models/turtlebot3_model/meshes/waffle_base.dae</uri>
               <scale>0.001 0.001 0.001</scale>
             </mesh>
@@ -43,5 +43,5 @@
           <always_on>true</always_on>
           <update_rate>200</update_rate>
-          <topic>$(arg namespace)/imu/data</topic>
+          <topic>$(arg namespace)/imu</topic>
           <gz_frame_id>imu_link</gz_frame_id>
           <imu>
@@ -89,30 +89,4 @@
         </sensor>
       </link>
-      <link name="gps_link">
-        <sensor name="navsat" type="navsat">
-          <always_on>true</always_on>
-          <update_rate>1</update_rate>
-          <topic>$(arg namespace)/gps/fix</topic>
-          <gz_frame_id>gps_link</gz_frame_id>
-          <navsat>
-            <position_sensing>
-              <horizontal>
-              <!-- Be carefull setting this.
-              Units in degree not in meters https://github.com/gazebosim/sdformat/issues/1572 -->
-                <noise type="gaussian">
-                  <mean>0.0</mean>
-                  <stddev>0.0</stddev>
-                </noise>
-              </horizontal>
-              <vertical>
-                <noise type="gaussian">
-                  <mean>0.0</mean>
-                  <stddev>0.0</stddev>
-                </noise>
-              </vertical>
-            </position_sensing>
-          </navsat>
-        </sensor>
-      </link>
       <link name="base_scan">
         <inertial>
@@ -141,10 +115,10 @@
           <geometry>
             <mesh>
-              <uri>package://demo_tb3/models/turtlebot3_model/meshes/lds.dae</uri>
+              <uri>package://demo_tb3_urdf/models/turtlebot3_model/meshes/lds.dae</uri>
               <scale>0.001 0.001 0.001</scale>
             </mesh>
           </geometry>
           <material>
-            <diffuse>0.5 0.5 0.5</diffuse>
+            <diffuse>1 1 1</diffuse>
           </material>
         </visual>
@@ -201,5 +175,5 @@
           <surface>
             <friction>
-              <bullet>
+              <ode>
                 <mu>1</mu>
                 <mu2>1</mu2>
@@ -207,8 +181,8 @@
                 <slip2>0</slip2>
                 <fdir1>0 0 1</fdir1>
-              </bullet>
+              </ode>
             </friction>
             <contact>
-              <bullet>
+              <ode>
                 <soft_cfm>0</soft_cfm>
                 <soft_erp>0.2</soft_erp>
@@ -217,5 +191,5 @@
                 <max_vel>0.01</max_vel>
                 <min_depth>0.001</min_depth>
-              </bullet>
+              </ode>
             </contact>
           </surface>
@@ -225,10 +199,10 @@
           <geometry>
             <mesh>
-              <uri>package://demo_tb3/models/turtlebot3_model/meshes/tire.dae</uri>
+              <uri>package://demo_tb3_urdf/models/turtlebot3_model/meshes/tire.dae</uri>
               <scale>0.001 0.001 0.001</scale>
             </mesh>
           </geometry>
           <material>
-            <diffuse>0.5 0.5 0.5</diffuse>
+            <diffuse>1 1 1</diffuse>
           </material>
         </visual>
@@ -257,5 +231,5 @@
           <surface>
             <friction>
-              <bullet>
+              <ode>
                 <mu>1</mu>
                 <mu2>1</mu2>
@@ -263,8 +237,8 @@
                 <slip2>0</slip2>
                 <fdir1>0 0 1</fdir1>
-              </bullet>
+              </ode>
             </friction>
             <contact>
-              <bullet>
+              <ode>
                 <soft_cfm>0</soft_cfm>
                 <soft_erp>0.2</soft_erp>
@@ -273,5 +247,5 @@
                 <max_vel>0.01</max_vel>
                 <min_depth>0.001</min_depth>
-              </bullet>
+              </ode>
             </contact>
           </surface>
@@ -281,15 +255,15 @@
           <geometry>
             <mesh>
-              <uri>package://demo_tb3/models/turtlebot3_model/meshes/tire.dae</uri>
+              <uri>package://demo_tb3_urdf/models/turtlebot3_model/meshes/tire.dae</uri>
               <scale>0.001 0.001 0.001</scale>
             </mesh>
           </geometry>
           <material>
-            <diffuse>0.5 0.5 0.5</diffuse>
+            <diffuse>1 1 1</diffuse>
           </material>
         </visual>
       </link>
       <link name='caster_back_right_link'>
-        <pose>-0.177 -0.064 -0.004 -1.57 0 0</pose>
+        <pose>-0.177 -0.064 -0.004 0 0 0</pose>
         <inertial>
           <mass>0.001</mass>
@@ -303,13 +277,13 @@
           </inertia>
         </inertial>
-        <collision name='caster_back_right_collision'>
+        <collision name='collision'>
           <geometry>
             <sphere>
-              <radius>0.0060000</radius>
+              <radius>0.006000</radius>
             </sphere>
           </geometry>
           <surface>
             <contact>
-              <bullet>
+              <ode>
                 <soft_cfm>0</soft_cfm>
                 <soft_erp>0.2</soft_erp>
@@ -318,41 +292,31 @@
                 <max_vel>0.01</max_vel>
                 <min_depth>0.001</min_depth>
-              </bullet>
+              </ode>
             </contact>
           </surface>
         </collision>
-        <visual name="sphere_visual">
+      </link>
+      <link name='caster_back_left_link'>
+        <pose>-0.177 0.064 -0.004 0 0 0</pose>
+        <inertial>
+          <mass>0.001</mass>
+          <inertia>
+            <ixx>0.00001</ixx>
+            <ixy>0.000</ixy>
+            <ixz>0.000</ixz>
+            <iyy>0.00001</iyy>
+            <iyz>0.000</iyz>
+            <izz>0.00001</izz>
+          </inertia>
+        </inertial>
+        <collision name='collision'>
           <geometry>
             <sphere>
-              <radius>0.0060000</radius>
-            </sphere>
-          </geometry>
-          <material>
-            <diffuse>0.5 0.5 0.5</diffuse>
-          </material>
-        </visual>
-      </link>
-      <link name='caster_back_left_link'>
-        <pose>-0.177 0.064 -0.004 -1.57 0 0</pose>
-        <inertial>
-          <mass>0.001</mass>
-          <inertia>
-            <ixx>0.00001</ixx>
-            <ixy>0.000</ixy>
-            <ixz>0.000</ixz>
-            <iyy>0.00001</iyy>
-            <iyz>0.000</iyz>
-            <izz>0.00001</izz>
-          </inertia>
-        </inertial>
-        <collision name='caster_back_left_collision'>
-          <geometry>
-            <sphere>
-              <radius>0.0060000</radius>
+              <radius>0.006000</radius>
             </sphere>
           </geometry>
           <surface>
             <contact>
-              <bullet>
+              <ode>
                 <soft_cfm>0</soft_cfm>
                 <soft_erp>0.2</soft_erp>
@@ -361,18 +325,8 @@
                 <max_vel>0.01</max_vel>
                 <min_depth>0.001</min_depth>
-              </bullet>
+              </ode>
             </contact>
           </surface>
         </collision>
-       <visual name="sphere_visual">
-          <geometry>
-            <sphere>
-              <radius>0.0060000</radius>
-            </sphere>
-          </geometry>
-          <material>
-            <diffuse>0.5 0.5 0.5</diffuse>
-          </material>
-        </visual>
       </link>
       <link name="camera_link">
@@ -475,18 +429,11 @@
         <pose>0.0 0 0.068 0 0 0</pose>
       </joint>
-      <joint name="gps_joint" type="fixed">
-        <parent>base_link</parent>
-        <child>gps_link</child>
-        <pose>-0.05 0 0.05 0 0 0</pose>
-      </joint>
       <plugin
         filename="gz-sim-diff-drive-system"
         name="gz::sim::systems::DiffDrive">
-        <!-- wheel information -->
         <left_joint>wheel_left_joint</left_joint>
         <right_joint>wheel_right_joint</right_joint>
         <wheel_separation>0.287</wheel_separation>
         <wheel_radius>0.033</wheel_radius>
-        <!-- limits -->
         <max_linear_acceleration>1</max_linear_acceleration>
         <min_linear_acceleration>-1</min_linear_acceleration>
@@ -497,7 +444,5 @@
         <max_angular_velocity>1.9</max_angular_velocity>
         <min_angular_velocity>-1.9</min_angular_velocity>
-        <!-- input -->
         <topic>$(arg namespace)/cmd_vel</topic>
-        <!-- output -->
         <odom_topic>$(arg namespace)/odom</odom_topic>
         <tf_topic>$(arg namespace)/tf</tf_topic>

File: ns_support_demo/demo_tb3_urdf/urdf/gz_waffle.urdf (robot description, URDF)
Before this commit: robot turtlebot3_waffle, 9 links, 8 joints
Links:
- link base_link: geometry collision box size=0.265 0.265 0.089; visual mesh filename=package://demo_tb3_urdf/models/turtlebot3_model/meshes/waff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 scale=0.001 0.001 0.001
- link base_scan: geometry collision cylinder length=0.055 radius=0.0508; visual mesh filename=package://demo_tb3_urdf/models/turtlebot3_model/meshes/lds.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 scale=0.001 0.001 0.001
- link wheel_left_link: geometry collision cylinder length=0.018 radius=0.033; visual mesh filename=package://demo_tb3_urdf/models/turtlebot3_model/meshes/tire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 scale=0.001 0.001 0.001
- link wheel_right_link: geometry collision cylinder length=0.018 radius=0.033; visual mesh filename=package://demo_tb3_urdf/models/turtlebot3_model/meshes/tire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 scale=0.001 0.001 0.001

File: ns_support_demo/demo_tb3_urdf/urdf/gz_waffle_gps.sdf.xacro (robot description, xacro)
@@ -2,5 +2,5 @@
 <sdf version="1.6" xmlns:xacro="http://www.ros.org/wiki/xacro">
     <xacro:arg name="namespace" default=""/>
-    <model name="turtlebot3_waffle">
+    <model name="turtlebot3_waffle_gps">
       <pose>0.0 0.0 0.0 0.0 0.0 0.0</pose>
       <link name="base_footprint"/>
@@ -30,5 +30,5 @@
           <geometry>
             <mesh>
-              <uri>package://demo_tb3/models/turtlebot3_model/meshes/waffle_base.dae</uri>
+              <uri>package://demo_tb3_urdf/models/turtlebot3_model/meshes/waffle_base.dae</uri>
               <scale>0.001 0.001 0.001</scale>
             </mesh>
@@ -43,5 +43,5 @@
           <always_on>true</always_on>
           <update_rate>200</update_rate>
-          <topic>$(arg namespace)/imu</topic>
+          <topic>$(arg namespace)/imu/data</topic>
           <gz_frame_id>imu_link</gz_frame_id>
           <imu>
@@ -89,4 +89,30 @@
         </sensor>
       </link>
+      <link name="gps_link">
+        <sensor name="navsat" type="navsat">
+          <always_on>true</always_on>
+          <update_rate>1</update_rate>
+          <topic>$(arg namespace)/gps/fix</topic>
+          <gz_frame_id>gps_link</gz_frame_id>
+          <navsat>
+            <position_sensing>
+              <horizontal>
+              <!-- Be carefull setting this.
+              Units in degree not in meters https://github.com/gazebosim/sdformat/issues/1572 -->
+                <noise type="gaussian">
+                  <mean>0.0</mean>
+                  <stddev>0.0</stddev>
+                </noise>
+              </horizontal>
+              <vertical>
+                <noise type="gaussian">
+                  <mean>0.0</mean>
+                  <stddev>0.0</stddev>
+                </noise>
+              </vertical>
+            </position_sensing>
+          </navsat>
+        </sensor>
+      </link>
       <link name="base_scan">
         <inertial>
@@ -115,10 +141,10 @@
           <geometry>
             <mesh>
-              <uri>package://demo_tb3/models/turtlebot3_model/meshes/lds.dae</uri>
+              <uri>package://demo_tb3_urdf/models/turtlebot3_model/meshes/lds.dae</uri>
               <scale>0.001 0.001 0.001</scale>
             </mesh>
           </geometry>
           <material>
-            <diffuse>1 1 1</diffuse>
+            <diffuse>0.5 0.5 0.5</diffuse>
           </material>
         </visual>
@@ -175,5 +201,5 @@
           <surface>
             <friction>
-              <ode>
+              <bullet>
                 <mu>1</mu>
                 <mu2>1</mu2>
@@ -181,8 +207,8 @@
                 <slip2>0</slip2>
                 <fdir1>0 0 1</fdir1>
-              </ode>
+              </bullet>
             </friction>
             <contact>
-              <ode>
+              <bullet>
                 <soft_cfm>0</soft_cfm>
                 <soft_erp>0.2</soft_erp>
@@ -191,5 +217,5 @@
                 <max_vel>0.01</max_vel>
                 <min_depth>0.001</min_depth>
-              </ode>
+              </bullet>
             </contact>
           </surface>
@@ -199,10 +225,10 @@
           <geometry>
             <mesh>
-              <uri>package://demo_tb3/models/turtlebot3_model/meshes/tire.dae</uri>
+              <uri>package://demo_tb3_urdf/models/turtlebot3_model/meshes/tire.dae</uri>
               <scale>0.001 0.001 0.001</scale>
             </mesh>
           </geometry>
           <material>
-            <diffuse>1 1 1</diffuse>
+            <diffuse>0.5 0.5 0.5</diffuse>
           </material>
         </visual>
@@ -231,5 +257,5 @@
           <surface>
             <friction>
-              <ode>
+              <bullet>
                 <mu>1</mu>
                 <mu2>1</mu2>
@@ -237,8 +263,8 @@
                 <slip2>0</slip2>
                 <fdir1>0 0 1</fdir1>
-              </ode>
+              </bullet>
             </friction>
             <contact>
-              <ode>
+              <bullet>
                 <soft_cfm>0</soft_cfm>
                 <soft_erp>0.2</soft_erp>
@@ -247,5 +273,5 @@
                 <max_vel>0.01</max_vel>
                 <min_depth>0.001</min_depth>
-              </ode>
+              </bullet>
             </contact>
           </surface>
@@ -255,15 +281,15 @@
           <geometry>
             <mesh>
-              <uri>package://demo_tb3/models/turtlebot3_model/meshes/tire.dae</uri>
+              <uri>package://demo_tb3_urdf/models/turtlebot3_model/meshes/tire.dae</uri>
               <scale>0.001 0.001 0.001</scale>
             </mesh>
           </geometry>
           <material>
-            <diffuse>1 1 1</diffuse>
+            <diffuse>0.5 0.5 0.5</diffuse>
           </material>
         </visual>
       </link>
       <link name='caster_back_right_link'>
-        <pose>-0.177 -0.064 -0.004 0 0 0</pose>
+        <pose>-0.177 -0.064 -0.004 -1.57 0 0</pose>
         <inertial>
           <mass>0.001</mass>
@@ -277,13 +303,13 @@
           </inertia>
         </inertial>
-        <collision name='collision'>
+        <collision name='caster_back_right_collision'>
           <geometry>
             <sphere>
-              <radius>0.006000</radius>
+              <radius>0.0060000</radius>
             </sphere>
           </geometry>
           <surface>
             <contact>
-              <ode>
+              <bullet>
                 <soft_cfm>0</soft_cfm>
                 <soft_erp>0.2</soft_erp>
@@ -292,11 +318,21 @@
                 <max_vel>0.01</max_vel>
                 <min_depth>0.001</min_depth>
-              </ode>
+              </bullet>
             </contact>
           </surface>
         </collision>
+        <visual name="sphere_visual">
+          <geometry>
+            <sphere>
+              <radius>0.0060000</radius>
+            </sphere>
+          </geometry>
+          <material>
+            <diffuse>0.5 0.5 0.5</diffuse>
+          </material>
+        </visual>
       </link>
       <link name='caster_back_left_link'>
-        <pose>-0.177 0.064 -0.004 0 0 0</pose>
+        <pose>-0.177 0.064 -0.004 -1.57 0 0</pose>
         <inertial>
           <mass>0.001</mass>
@@ -310,13 +346,13 @@
           </inertia>
         </inertial>
-        <collision name='collision'>
+        <collision name='caster_back_left_collision'>
           <geometry>
             <sphere>
-              <radius>0.006000</radius>
+              <radius>0.0060000</radius>
             </sphere>
           </geometry>
           <surface>
             <contact>
-              <ode>
+              <bullet>
                 <soft_cfm>0</soft_cfm>
                 <soft_erp>0.2</soft_erp>
@@ -325,8 +361,18 @@
                 <max_vel>0.01</max_vel>
                 <min_depth>0.001</min_depth>
-              </ode>
+              </bullet>
             </contact>
           </surface>
         </collision>
+       <visual name="sphere_visual">
+          <geometry>
+            <sphere>
+              <radius>0.0060000</radius>
+            </sphere>
+          </geometry>
+          <material>
+            <diffuse>0.5 0.5 0.5</diffuse>
+          </material>
+        </visual>
       </link>
       <link name="camera_link">
@@ -429,11 +475,18 @@
         <pose>0.0 0 0.068 0 0 0</pose>
       </joint>
+      <joint name="gps_joint" type="fixed">
+        <parent>base_link</parent>
+        <child>gps_link</child>
+        <pose>-0.05 0 0.05 0 0 0</pose>
+      </joint>
       <plugin
         filename="gz-sim-diff-drive-system"
         name="gz::sim::systems::DiffDrive">
+        <!-- wheel information -->
         <left_joint>wheel_left_joint</left_joint>
         <right_joint>wheel_right_joint</right_joint>
         <wheel_separation>0.287</wheel_separation>
         <wheel_radius>0.033</wheel_radius>
+        <!-- limits -->
         <max_linear_acceleration>1</max_linear_acceleration>
         <min_linear_acceleration>-1</min_linear_acceleration>
@@ -444,5 +497,7 @@
         <max_angular_velocity>1.9</max_angular_velocity>
         <min_angular_velocity>-1.9</min_angular_velocity>
+        <!-- input -->
         <topic>$(arg namespace)/cmd_vel</topic>
+        <!-- output -->
         <odom_topic>$(arg namespace)/odom</odom_topic>
         <tf_topic>$(arg namespace)/tf</tf_topic>

File: ns_support_demo/demo_tb3_urdf/urdf/gz_waffle_gps.urdf (robot description, URDF)
Before this commit: robot turtlebot3_waffle_gps, 10 links, 9 joints
Links:
- link base_link: geometry collision box size=0.265 0.265 0.089; visual mesh filename=package://demo_tb3_urdf/models/turtlebot3_model/meshes/waff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 scale=0.001 0.001 0.001
- link base_scan: geometry collision cylinder length=0.055 radius=0.0508; visual mesh filename=package://demo_tb3_urdf/models/turtlebot3_model/meshes/lds.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 scale=0.001 0.001 0.001
- link wheel_left_link: geometry collision cylinder length=0.018 radius=0.033; visual mesh filename=package://demo_tb3_urdf/models/turtlebot3_model/meshes/tire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 scale=0.001 0.001 0.001
- link wheel_right_link: geometry collision cylinder length=0.018 radius=0.033; visual mesh filename=package://demo_tb3_urdf/models/turtlebot3_model/meshes/tire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 scale=0.001 0.001 0.001
